Commit message: Set sensible limits for missing joint limits in urdf

File: public/urdf/cassie/cassie.urdf (robot description, URDF)
Before this commit: robot cassie, 23 links, 22 joints
Joints:
- joint ankle_joint_left: limit lower=-100 upper=100 effort=0 velocity=100 -> lower=1 upper=2.8 effort=0 velocity=100
- joint ankle_joint_right: limit lower=-100 upper=100 effort=0 velocity=100 -> lower=1 upper=2.8 effort=0 velocity=100
- joint knee_to_shin_left: limit lower=-100 upper=100 effort=0 velocity=100 -> lower=-0.6 upper=0 effort=0 velocity=100
- joint knee_to_shin_right: limit lower=-100 upper=100 effort=0 velocity=100 -> lower=-0.6 upper=0 effort=0 velocity=100

File: public/urdf/so-100/so_100.urdf (robot description, URDF)
Before this commit: robot so_100, 7 links, 6 joints
Joints:
- joint Elbow: limit (none) -> lower=-0.8 upper=2.3 effort=10.0 velocity=5.0
- joint Gripper: limit (none) -> lower=0 upper=1.7 effort=2.0 velocity=2.0
- joint Shoulder_Pitch: limit (none) -> lower=-2 upper=1.57 effort=10.0 velocity=5.0
- joint Shoulder_Rotation: limit (none) -> lower=-1.5708 upper=1.5708 effort=10.0 velocity=5.0
- joint Wrist_Pitch: limit (none) -> lower=-1.5 upper=0.8 effort=5.0 velocity=3.0
- joint Wrist_Roll: limit (none) -> lower=-3.14159 upper=3.14159 effort=5.0 velocity=3.0
